File: serendipboard_v2.sch (EAGLE design)
At the start: 45 parts, among them IC1 TP4056, IC2 DW01A, IC3 DS3231/SO, Q1 FS8205A, Q2 DMP3056LSD, Q3 20V/0.2A/8MHz/1.2Ω/1Vth, Q4 20V/0.2A/8MHz/1.2Ω/1Vth, U1 MAX17043, U2 AP2112-3.3, U3 AP2112-3.3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

Commit message: Update serendipboard_v2.sch
Parts:
- added C16: 10uF, rcl:C-EUC0805
- added C17: 1uF, rcl:C-EUC0805
- added J2: (no value), SparkFun-Connectors:CONN_02
- added Q5, Q6: 600mA/40V, SparkFun-DiscreteSemi:TRANS_NPN-MMBT2222AL
- added R13, R14, R15, R16: 1k, rcl:R-US_R0805
Connections:
- new net BATT_MONITOR: C17.1, R15.2, R16.2
- new net BUZZER: R14.1
- new net MOTOR: R13.1
- new net N$13: Q5.B, R13.2
- new net N$14: Q6.B, R14.2
- new net N$17: J2.1, Q5.C
- net GND: now also C16.2, C17.2, Q5.E, Q6.E, R16.1
- net VCC: now also C16.1, J2.2, R15.1
Other:
- note added: "Buzzer"
- note added: "Motor"
- note added: "Voltage Monitoring"
- note removed: "battery_conn"
- note removed: "buzzer"
- note removed: "motor"
- moved on the sheet: J1

Commit message: Update serendipboard_v2.sch
Parts:
- added R17: 10k, rcl:R-US_R0805
- added R18, R19, R20: 20k, rcl:R-US_R0805
- Q6: value 600mA/40V -> TRANS_NPN-MMBT2222AL
Connections:
- new net CHARGER: R17.1, R18.2
- net GND: now also R18.1
- net SCL: now also R20.1
- net SDA: now also R19.1
- net VCC: now also R17.2, R19.2, R20.2
Other:
- note added: "Charger Detection"
- note added: "I2C Pullups"
- moved on the sheet: C16, C17, C8, C9, CN1, J2, Q3, Q5, Q6, R11, R13, R14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

Commit message: Update serendipboard_v2.sch
Other:
- note added: "buscar buzzer"
- moved on the sheet: J2, Q5, R13
Changed lines of the file:
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@@
 <text x="157.48" y="27.94" size="1.778" layer="94" rot="R180">Battery Connector</text>
 <wire x1="134.62" y1="35.56" x2="134.62" y2="0" width="0.1524" layer="94" style="shortdash"/>
-<text x="35.56" y="91.44" size="1.778" layer="94" rot="R180">Motor</text>
+<text x="27.94" y="91.44" size="1.778" layer="94" rot="R180">Motor</text>
 <text x="111.76" y="91.44" size="1.778" layer="94" rot="R180">Voltage Monitoring</text>
 <text x="30.48" y="43.18" size="1.778" layer="94" rot="R180">Buzzer</text>
@@
 <wire x1="0" y1="48.26" x2="50.8" y2="48.26" width="0.1524" layer="94" style="shortdash"/>
 <text x="81.28" y="43.18" size="1.778" layer="94" rot="R180">Charger Detection</text>
-<wire x1="50.8" y1="48.26" x2="66.04" y2="48.26" width="0.1524" layer="94" style="shortdash"/>
-<wire x1="66.04" y1="48.26" x2="88.9" y2="48.26" width="0.1524" layer="94" style="shortdash"/>
+<wire x1="50.8" y1="48.26" x2="88.9" y2="48.26" width="0.1524" layer="94" style="shortdash"/>
 <wire x1="88.9" y1="48.26" x2="134.62" y2="48.26" width="0.1524" layer="94" style="shortdash"/>
-<wire x1="66.04" y1="96.52" x2="66.04" y2="48.26" width="0.1524" layer="94" style="shortdash"/>
 <wire x1="88.9" y1="48.26" x2="88.9" y2="0" width="0.1524" layer="94" style="shortdash"/>
 <wire x1="50.8" y1="48.26" x2="50.8" y2="0" width="0.1524" layer="94" style="shortdash"/>
 <text x="119.38" y="43.18" size="1.778" layer="94" rot="R180">I2C Pullups</text>
+<text x="27.94" y="25.4" size="1.778" layer="95">buscar buzzer</text>
 </plain>
 <instances>
@@
 <attribute name="VALUE" x="154.94" y="20.32" size="1.27" layer="96" rot="R180"/>
 </instance>
-<instance part="Q5" gate="G$1" x="38.1" y="68.58" smashed="yes">
-<attribute name="NAME" x="40.64" y="68.58" size="1.778" layer="95" font="vector"/>
-<attribute name="VALUE" x="40.64" y="66.294" size="1.778" layer="96" font="vector"/>
+<instance part="Q5" gate="G$1" x="30.48" y="68.58" smashed="yes">
+<attribute name="NAME" x="33.02" y="68.58" size="1.778" layer="95" font="vector"/>
+<attribute name="VALUE" x="33.02" y="66.294" size="1.778" layer="96" font="vector"/>
 </instance>
 <instance part="Q6" gate="G$1" x="30.48" y="17.78" smashed="yes">
@@
 <attribute name="VALUE" x="33.02" y="15.494" size="1.778" layer="96" font="vector"/>
 </instance>
-<instance part="R13" gate="G$1" x="27.94" y="68.58" smashed="yes">
-<attribute name="NAME" x="24.13" y="70.0786" size="1.778" layer="95"/>
-<attribute name="VALUE" x="24.13" y="65.278" size="1.778" layer="96"/>
+<instance part="R13" gate="G$1" x="20.32" y="68.58" smashed="yes">
+<attribute name="NAME" x="16.51" y="70.0786" size="1.778" layer="95"/>
+<attribute name="VALUE" x="16.51" y="65.278" size="1.778" layer="96"/>
 </instance>
 <instance part="R14" gate="G$1" x="20.32" y="17.78" smashed="yes">
@@
 <attribute name="VALUE" x="16.51" y="14.478" size="1.778" layer="96"/>
 </instance>
-<instance part="GND29" gate="1" x="40.64" y="58.42" smashed="yes">
-<attribute name="VALUE" x="38.1" y="55.88" size="1.778" layer="96"/>
+<instance part="GND29" gate="1" x="33.02" y="58.42" smashed="yes">
+<attribute name="VALUE" x="30.48" y="55.88" size="1.778" layer="96"/>
 </instance>
 <instance part="GND30" gate="1" x="33.02" y="7.62" smashed="yes">
 <attribute name="VALUE" x="30.48" y="5.08" size="1.778" layer="96"/>
 </instance>
-<instance part="P+23" gate="VCC" x="40.64" y="83.82" smashed="yes">
-<attribute name="VALUE" x="43.18" y="86.36" size="1.27" layer="96" rot="R180"/>
+<instance part="P+23" gate="VCC" x="33.02" y="83.82" smashed="yes">
+<attribute name="VALUE" x="35.56" y="86.36" size="1.27" layer="96" rot="R180"/>
 </instance>
 <instance part="P+24" gate="VCC" x="33.02" y="33.02" smashed="yes">
 <attribute name="VALUE" x="35.56" y="35.56" size="1.27" layer="96" rot="R180"/>
 </instance>
-<instance part="J2" gate="G$1" x="50.8" y="76.2" smashed="yes" rot="MR0">
-<attribute name="VALUE" x="53.34" y="71.374" size="1.778" layer="96" font="vector" rot="MR0"/>
-<attribute name="NAME" x="53.34" y="81.788" size="1.778" layer="95" font="vector" rot="MR0"/>
+<instance part="J2" gate="G$1" x="43.18" y="76.2" smashed="yes" rot="MR0">
+<attribute name="VALUE" x="45.72" y="71.374" size="1.778" layer="96" font="vector" rot="MR0"/>
+<attribute name="NAME" x="45.72" y="81.788" size="1.778" layer="95" font="vector" rot="MR0"/>
 </instance>
 <instance part="R15" gate="G$1" x="93.98" y="76.2" smashed="yes">
@@
 <pinref part="GND29" gate="1" pin="GND"/>
 <pinref part="Q5" gate="G$1" pin="E"/>
-<wire x1="40.64" y1="60.96" x2="40.64" y2="63.5" width="0.1524" layer="91"/>
+<wire x1="33.02" y1="60.96" x2="33.02" y2="63.5" width="0.1524" layer="91"/>
 </segment>
 <segment>
@@
 <pinref part="J2" gate="G$1" pin="2"/>
 <pinref part="P+23" gate="VCC" pin="VCC"/>
-<wire x1="43.18" y1="78.74" x2="40.64" y2="78.74" width="0.1524" layer="91"/>
-<wire x1="40.64" y1="78.74" x2="40.64" y2="81.28" width="0.1524" layer="91"/>
+<wire x1="35.56" y1="78.74" x2="33.02" y2="78.74" width="0.1524" layer="91"/>
+<wire x1="33.02" y1="78.74" x2="33.02" y2="81.28" width="0.1524" layer="91"/>
 </segment>
 <segment>
@@
 <pinref part="R13" gate="G$1" pin="2"/>
 <pinref part="Q5" gate="G$1" pin="B"/>
-<wire x1="33.02" y1="68.58" x2="35.56" y2="68.58" width="0.1524" layer="91"/>
+<wire x1="25.4" y1="68.58" x2="27.94" y2="68.58" width="0.1524" layer="91"/>
 </segment>
 </net>
@@
 <segment>
 <pinref part="R13" gate="G$1" pin="1"/>
-<wire x1="22.86" y1="68.58" x2="20.32" y2="68.58" width="0.1524" layer="91"/>
-<label x="20.32" y="68.58" size="1.27" layer="95" rot="R180" xref="yes"/>
+<wire x1="15.24" y1="68.58" x2="12.7" y2="68.58" width="0.1524" layer="91"/>
+<label x="12.7" y="68.58" size="1.27" layer="95" rot="R180" xref="yes"/>
 </segment>
 </net>
@@
 <pinref part="Q5" gate="G$1" pin="C"/>
 <pinref part="J2" gate="G$1" pin="1"/>
-<wire x1="40.64" y1="73.66" x2="40.64" y2="76.2" width="0.1524" layer="91"/>
-<wire x1="40.64" y1="76.2" x2="43.18" y2="76.2" width="0.1524" layer="91"/>
-</segment>
-</net>
+<wire x1="33.02" y1="73.66" x2="33.02" y2="76.2" width="0.1524" layer="91"/>
+<wire x1="33.02" y1="76.2" x2="35.56" y2="76.2" width="0.1524" layer="91"/>
+</segment>
+</net>

Commit message: Update serendipboard_v2.sch
Parts:
- removed CN1: (no value), adafruit:USBMINIB
- added J3: (no value), SparkFun-Connectors:CONN_04PTH
Connections:
- net GND: now also J3.3
- net SCL: now also J3.1
- net SDA: now also J3.2
- net VCC: now also J3.4
Other:
- note added: "Oled"
- moved on the sheet: B1, C10, C11, C16, C17, IC3, J2, Q5, R13, R15, R16, U3

Commit message: Update serendipboard_v2.sch
Parts:
- added U5: ESP32-WROOM-32D, ESP32-WROOM-32D:ESP32-WROOM-32D
Changed lines of the file:
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@@
 <part name="P+8" library="supply1" library_urn="urn:adsk.eagle:library:371" deviceset="VCC" device="" value="3.3Vesp"/>
 <part name="P+9" library="supply1" library_urn="urn:adsk.eagle:library:371" deviceset="VCC" device="" value="VIN"/>
+<part name="U5" library="ESP32-WROOM-32D" library_urn="urn:adsk.eagle:library:27379448" deviceset="ESP32-WROOM-32D" device="" package3d_urn="urn:adsk.eagle:package:27379451/1"/>
 </parts>
 <sheets>
@@
 <attribute name="NAME" x="155.448" y="149.098" size="1.778" layer="95" rot="R180"/>
 </instance>
-<instance part="Q2" gate="B" x="165.1" y="187.96" smashed="yes" rot="R270">
-<attribute name="VALUE" x="170.18" y="187.452" size="1.778" layer="96" align="top-left"/>
-<attribute name="NAME" x="170.18" y="188.468" size="1.778" layer="95"/>
-</instance>
 <instance part="R4" gate="G$1" x="162.56" y="170.18" smashed="yes" rot="R180">
 <attribute name="NAME" x="166.37" y="168.6814" size="1.778" layer="95" rot="R180"/>
@@
 <attribute name="VALUE" x="15.24" y="167.64" size="1.27" layer="96" rot="R180"/>
 </instance>
+<instance part="U5" gate="G$1" x="124.46" y="137.16" smashed="yes">
+<attribute name="NAME" x="109.4241" y="168.7545" size="1.778" layer="95"/>
+<attribute name="VALUE" x="109.1733" y="101.4919" size="1.778" layer="96"/>
+</instance>
 </instances>

Commit message: Update serendipboard_v2.sch
Parts:
- added C18: 10uF, rcl:C-EUC0805
- added J4: USB_MINI, SparkFun-Connectors:USB_MINI-B_SMT
- added Q7: (no value), SparkFun-DiscreteSemi:TRANS_PNP_DUALSOT-363
- added R21, R22, R23: 1k, rcl:R-US_R0805
- added U6: CP2102N, SparkFun-IC-Comms:CP2102N
Connections:
- new net D+: J4.D+
- new net D-: J4.D-
- new net N$15: U6.D-
- new net N$16: U6.D+
- new net N$18: U6.VBUS
- new net N$19: U6.VREGIN
- net GND: now also J4.GND
- net VCC: now also J4.VBUS
Other:
- moved on the sheet: U5
Changed lines of the file:
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@@
 <part name="P+9" library="supply1" library_urn="urn:adsk.eagle:library:371" deviceset="VCC" device="" value="VIN"/>
 <part name="U5" library="ESP32-WROOM-32D" library_urn="urn:adsk.eagle:library:27379448" deviceset="ESP32-WROOM-32D" device="" package3d_urn="urn:adsk.eagle:package:27379451/1"/>
+<part name="U6" library="SparkFun-IC-Comms" deviceset="CP2102N" device=""/>
+<part name="J4" library="SparkFun-Connectors" deviceset="USB_MINI-B" device="_SMT" value="USB_MINI"/>
+<part name="R21" library="rcl" library_urn="urn:adsk.eagle:library:334" deviceset="R-US_" device="R0805" package3d_urn="urn:adsk.eagle:package:23553/2" value="1k"/>
+<part name="C18" library="rcl" library_urn="urn:adsk.eagle:library:334" deviceset="C-EU" device="C0805" package3d_urn="urn:adsk.eagle:package:23617/2" value="10uF"/>
+<part name="GND36" library="supply1" library_urn="urn:adsk.eagle:library:371" deviceset="GND" device=""/>
+<part name="P+29" library="supply1" library_urn="urn:adsk.eagle:library:371" deviceset="VCC" device="" value="VBUS"/>
+<part name="Q7" library="SparkFun-DiscreteSemi" deviceset="TRANS_PNP_DUAL" device="SOT-363" package3d_urn="urn:adsk.eagle:package:29757/2"/>
+<part name="R22" library="rcl" library_urn="urn:adsk.eagle:library:334" deviceset="R-US_" device="R0805" package3d_urn="urn:adsk.eagle:package:23553/2" value="1k"/>
+<part name="R23" library="rcl" library_urn="urn:adsk.eagle:library:334" deviceset="R-US_" device="R0805" package3d_urn="urn:adsk.eagle:package:23553/2" value="1k"/>
 </parts>
 <sheets>
@@
 <attribute name="VALUE" x="15.24" y="167.64" size="1.27" layer="96" rot="R180"/>
 </instance>
-<instance part="U5" gate="G$1" x="124.46" y="137.16" smashed="yes">
-<attribute name="NAME" x="109.4241" y="168.7545" size="1.778" layer="95"/>
-<attribute name="VALUE" x="109.1733" y="101.4919" size="1.778" layer="96"/>
+<instance part="U5" gate="G$1" x="33.02" y="50.8" smashed="yes">
+<attribute name="NAME" x="17.9841" y="82.3945" size="1.778" layer="95"/>
+<attribute name="VALUE" x="17.7333" y="15.1319" size="1.778" layer="96"/>
+</instance>
+<instance part="U6" gate="G$1" x="226.06" y="149.86" smashed="yes">
+<attribute name="NAME" x="208.28" y="172.974" size="1.778" layer="95"/>
+<attribute name="VALUE" x="208.28" y="124.46" size="1.778" layer="96"/>
+</instance>
+<instance part="J4" gate="G$1" x="134.62" y="152.4" smashed="yes">
+<attribute name="VALUE" x="129.54" y="142.494" size="1.778" layer="96" font="vector" rot="MR180" align="top-left"/>
+<attribute name="NAME" x="132.08" y="162.814" size="1.778" layer="95" font="vector"/>
+</instance>
+<instance part="R21" gate="G$1" x="165.1" y="127" smashed="yes">
+<attribute name="NAME" x="161.29" y="128.4986" size="1.778" layer="95"/>
+<attribute name="VALUE" x="161.29" y="123.698" size="1.778" layer="96"/>
+</instance>
+<instance part="C18" gate="G$1" x="177.8" y="114.3" smashed="yes" rot="MR0">
+<attribute name="NAME" x="176.276" y="114.681" size="1.778" layer="95" rot="MR0"/>
+<attribute name="VALUE" x="176.276" y="109.601" size="1.778" layer="96" rot="MR0"/>
+</instance>
+<instance part="GND36" gate="1" x="144.78" y="144.78" smashed="yes">
+<attribute name="VALUE" x="142.24" y="142.24" size="1.27" layer="96"/>
+</instance>
+<instance part="P+29" gate="VCC" x="144.78" y="162.56" smashed="yes">
+<attribute name="VALUE" x="147.32" y="165.1" size="1.27" layer="96" rot="R180"/>
+</instance>
+<instance part="Q7" gate="G$1" x="175.26" y="86.36" smashed="yes" rot="MR180">
+<attribute name="NAME" x="177.8" y="86.36" size="1.778" layer="95" font="vector" rot="MR180"/>
+<attribute name="VALUE" x="177.8" y="86.614" size="1.778" layer="96" font="vector" rot="MR180" align="top-left"/>
+</instance>
+<instance part="Q7" gate="G$2" x="175.26" y="66.04" smashed="yes">
+<attribute name="NAME" x="177.8" y="66.04" size="1.778" layer="95" font="vector"/>
+<attribute name="VALUE" x="177.8" y="65.786" size="1.778" layer="96" font="vector" align="top-left"/>
+</instance>
+<instance part="R22" gate="G$1" x="165.1" y="86.36" smashed="yes">
+<attribute name="NAME" x="161.29" y="87.8586" size="1.778" layer="95"/>
+<attribute name="VALUE" x="161.29" y="83.058" size="1.778" layer="96"/>
+</instance>
+<instance part="R23" gate="G$1" x="165.1" y="66.04" smashed="yes">
+<attribute name="NAME" x="161.29" y="67.5386" size="1.778" layer="95"/>
+<attribute name="VALUE" x="161.29" y="62.738" size="1.778" layer="96"/>
 </instance>
 </instances>
@@
 <pinref part="GND16" gate="1" pin="GND"/>
 <pinref part="C9" gate="G$1" pin="2"/>
+</segment>
+<segment>
+<pinref part="J4" gate="G$1" pin="GND"/>
+<wire x1="139.7" y1="149.86" x2="144.78" y2="149.86" width="0.1524" layer="91"/>
+<wire x1="144.78" y1="149.86" x2="144.78" y2="147.32" width="0.1524" layer="91"/>
+<pinref part="GND36" gate="1" pin="GND"/>
 </segment>
 </net>
@@
 <pinref part="P+9" gate="VCC" pin="VCC"/>
 </segment>
+<segment>
+<pinref part="J4" gate="G$1" pin="VBUS"/>
+<wire x1="139.7" y1="160.02" x2="144.78" y2="160.02" width="0.1524" layer="91"/>
+<pinref part="P+29" gate="VCC" pin="VCC"/>
+</segment>
 </net>
 <net name="N$8" class="0">
@@
 </segment>
 </net>
+<net name="D-" class="0">
+<segment>
+<pinref part="J4" gate="G$1" pin="D-"/>
+<wire x1="139.7" y1="157.48" x2="142.24" y2="157.48" width="0.1524" layer="91"/>
+<label x="142.24" y="157.48" size="1.27" layer="95" xref="yes"/>
+</segment>
+</net>
+<net name="D+" class="0">
+<segment>
+<pinref part="J4" gate="G$1" pin="D+"/>
+<wire x1="139.7" y1="154.94" x2="142.24" y2="154.94" width="0.1524" layer="91"/>
+<label x="142.24" y="154.94" size="1.27" layer="95" xref="yes"/>
+</segment>
+</net>
+<net name="N$15" class="0">
+<segment>
+<pinref part="U6" gate="G$1" pin="D-"/>
+<wire x1="205.74" y1="147.32" x2="203.2" y2="147.32" width="0.1524" layer="91"/>
+</segment>
+</net>
+<net name="N$16" class="0">
+<segment>
+<pinref part="U6" gate="G$1" pin="D+"/>
+<wire x1="205.74" y1="149.86" x2="203.2" y2="149.86" width="0.1524" layer="91"/>
+</segment>
+</net>
+<net name="N$18" class="0">
+<segment>
+<pinref part="U6" gate="G$1" pin="VBUS"/>
+<wire x1="205.74" y1="152.4" x2="203.2" y2="152.4" width="0.1524" layer="91"/>
+</segment>
+</net>
+<net name="N$19" class="0">
+<segment>
+<pinref part="U6" gate="G$1" pin="VREGIN"/>
+<wire x1="205.74" y1="154.94" x2="203.2" y2="154.94" width="0.1524" layer="91"/>
+</segment>
+</net>

Commit message: Update serendipboard_v2.sch
Parts:
- added U7: CP2102N-A01-GQFN28, CP2102N-A01-GQFN28:CP2102N-A01-GQFN28
Connections:
- removed net N$15: U6.D-
- removed net N$16: U6.D+
- removed net N$18: U6.VBUS
- removed net N$19: U6.VREGIN
Other:
- moved on the sheet: U6
Changed lines of the file:
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@@
 <part name="R22" library="rcl" library_urn="urn:adsk.eagle:library:334" deviceset="R-US_" device="R0805" package3d_urn="urn:adsk.eagle:package:23553/2" value="1k"/>
 <part name="R23" library="rcl" library_urn="urn:adsk.eagle:library:334" deviceset="R-US_" device="R0805" package3d_urn="urn:adsk.eagle:package:23553/2" value="1k"/>
+<part name="U7" library="CP2102N-A01-GQFN28" deviceset="CP2102N-A01-GQFN28" device=""/>
 </parts>
 <sheets>
@@
 <attribute name="VALUE" x="17.7333" y="15.1319" size="1.778" layer="96"/>
 </instance>
-<instance part="U6" gate="G$1" x="226.06" y="149.86" smashed="yes">
-<attribute name="NAME" x="208.28" y="172.974" size="1.778" layer="95"/>
-<attribute name="VALUE" x="208.28" y="124.46" size="1.778" layer="96"/>
+<instance part="U6" gate="G$1" x="220.98" y="149.86" smashed="yes">
+<attribute name="NAME" x="203.2" y="172.974" size="1.778" layer="95"/>
+<attribute name="VALUE" x="203.2" y="124.46" size="1.778" layer="96"/>
 </instance>
 <instance part="J4" gate="G$1" x="134.62" y="152.4" smashed="yes">
@@
 <attribute name="NAME" x="161.29" y="67.5386" size="1.778" layer="95"/>
 <attribute name="VALUE" x="161.29" y="62.738" size="1.778" layer="96"/>
+</instance>
+<instance part="U7" gate="G$1" x="96.52" y="114.3" smashed="yes" rot="MR0">
+<attribute name="NAME" x="114.3568" y="145.3839" size="1.6829" layer="95" rot="MR0"/>
+<attribute name="VALUE" x="114.3288" y="81.227" size="1.679509375" layer="96" rot="MR0"/>
 </instance>
 </instances>
@@
 </segment>
 </net>
-<net name="N$15" class="0">
-<segment>
-<pinref part="U6" gate="G$1" pin="D-"/>
-<wire x1="205.74" y1="147.32" x2="203.2" y2="147.32" width="0.1524" layer="91"/>
-</segment>
-</net>
-<net name="N$16" class="0">
-<segment>
-<pinref part="U6" gate="G$1" pin="D+"/>
-<wire x1="205.74" y1="149.86" x2="203.2" y2="149.86" width="0.1524" layer="91"/>
-</segment>
-</net>
-<net name="N$18" class="0">
-<segment>
-<pinref part="U6" gate="G$1" pin="VBUS"/>
-<wire x1="205.74" y1="152.4" x2="203.2" y2="152.4" width="0.1524" layer="91"/>
-</segment>
-</net>
-<net name="N$19" class="0">
-<segment>
-<pinref part="U6" gate="G$1" pin="VREGIN"/>
-<wire x1="205.74" y1="154.94" x2="203.2" y2="154.94" width="0.1524" layer="91"/>
-</segment>
-</net>

Commit message: Update serendipboard_v2.sch
Parts:
- removed U6: CP2102N, SparkFun-IC-Comms:CP2102N
Other:
- moved on the sheet: C18, U5, U7
Changed lines of the file:
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@@
 <part name="P+9" library="supply1" library_urn="urn:adsk.eagle:library:371" deviceset="VCC" device="" value="VIN"/>
 <part name="U5" library="ESP32-WROOM-32D" library_urn="urn:adsk.eagle:library:27379448" deviceset="ESP32-WROOM-32D" device="" package3d_urn="urn:adsk.eagle:package:27379451/1"/>
-<part name="U6" library="SparkFun-IC-Comms" deviceset="CP2102N" device=""/>
 <part name="J4" library="SparkFun-Connectors" deviceset="USB_MINI-B" device="_SMT" value="USB_MINI"/>
 <part name="R21" library="rcl" library_urn="urn:adsk.eagle:library:334" deviceset="R-US_" device="R0805" package3d_urn="urn:adsk.eagle:package:23553/2" value="1k"/>
@@
 <attribute name="VALUE" x="15.24" y="167.64" size="1.27" layer="96" rot="R180"/>
 </instance>
-<instance part="U5" gate="G$1" x="33.02" y="50.8" smashed="yes">
-<attribute name="NAME" x="17.9841" y="82.3945" size="1.778" layer="95"/>
-<attribute name="VALUE" x="17.7333" y="15.1319" size="1.778" layer="96"/>
-</instance>
-<instance part="U6" gate="G$1" x="220.98" y="149.86" smashed="yes">
-<attribute name="NAME" x="203.2" y="172.974" size="1.778" layer="95"/>
-<attribute name="VALUE" x="203.2" y="124.46" size="1.778" layer="96"/>
+<instance part="U5" gate="G$1" x="48.26" y="83.82" smashed="yes">
+<attribute name="NAME" x="33.2241" y="115.4145" size="1.778" layer="95"/>
+<attribute name="VALUE" x="32.9733" y="48.1519" size="1.778" layer="96"/>
 </instance>
 <instance part="J4" gate="G$1" x="134.62" y="152.4" smashed="yes">
@@
 <attribute name="VALUE" x="161.29" y="123.698" size="1.778" layer="96"/>
 </instance>
-<instance part="C18" gate="G$1" x="177.8" y="114.3" smashed="yes" rot="MR0">
-<attribute name="NAME" x="176.276" y="114.681" size="1.778" layer="95" rot="MR0"/>
-<attribute name="VALUE" x="176.276" y="109.601" size="1.778" layer="96" rot="MR0"/>
+<instance part="C18" gate="G$1" x="182.88" y="129.54" smashed="yes" rot="MR0">
+<attribute name="NAME" x="181.356" y="129.921" size="1.778" layer="95" rot="MR0"/>
+<attribute name="VALUE" x="181.356" y="124.841" size="1.778" layer="96" rot="MR0"/>
 </instance>
 <instance part="GND36" gate="1" x="144.78" y="144.78" smashed="yes">
@@
 <attribute name="VALUE" x="161.29" y="62.738" size="1.778" layer="96"/>
 </instance>
-<instance part="U7" gate="G$1" x="96.52" y="114.3" smashed="yes" rot="MR0">
-<attribute name="NAME" x="114.3568" y="145.3839" size="1.6829" layer="95" rot="MR0"/>
-<attribute name="VALUE" x="114.3288" y="81.227" size="1.679509375" layer="96" rot="MR0"/>
+<instance part="U7" gate="G$1" x="231.14" y="142.24" smashed="yes" rot="MR0">
+<attribute name="NAME" x="248.9768" y="173.3239" size="1.6829" layer="95" rot="MR0"/>
+<attribute name="VALUE" x="248.9488" y="109.167" size="1.679509375" layer="96" rot="MR0"/>
 </instance>
 </instances>
