File: serendipboard_v2.sch (EAGLE design)
At the start: 83 parts, among them IC1 TP4056, IC2 DW01A, IC3 DS3231/SO, J4 USB_MINI, Q1 FS8205A, Q3 RUC002N05HZGT116, Q4 DMG3415U, Q5 600mA/40V, Q6 TRANS_NPN-MMBT2222AL, Q7 RUC002N05HZGT116, U1 MAX17043, U2 AP2112-3.3, U3 AP2112-3.3, U4 9DoF IMU, U5 ESP32-WROOM-32D, U6 FT231XQ-R

Commit message: Update serendipboard_v2.sch
Parts:
- IC1: WEBLINK (none) -> https://lcsc.com/product-detail/PMIC-Battery-Management_UMW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
- IC2: WEBLINK (none) -> https://lcsc.com/product-detail/Battery-Protection-ICs_PUOL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
- IC3: WEBLINK (none) -> https://www.mouser.com/ProductDetail/Maxim-Integrated/DS323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
- LS1: WEBLINK (none) -> https://www.mouser.com/ProductDetail/CUI-Devices/CST-931AP?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
- Q1: WEBLINK (none) -> https://lcsc.com/product-detail/MOSFET_FUXINSEMI-FS8205A_C9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
- U1: WEBLINK (none) -> https://www.mouser.com/ProductDetail/Maxim-Integrated/MAX17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
- U4: WEBLINK (none) -> https://www.mouser.com/ProductDetail/TDK-InvenSense/ICM-209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
- U5: WEBLINK (none) -> https://www.mouser.com/ProductDetail/Espressif-Systems/ESP3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
Changed lines of the file:
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@@
 </classes>
 <parts>
-<part name="IC1" library="TP4056" deviceset="TP4056" device=""/>
-<part name="Q1" library="FS8205A" deviceset="FS8205A" device=""/>
-<part name="IC2" library="DW01A" deviceset="DW01A" device=""/>
+<part name="IC1" library="TP4056" deviceset="TP4056" device="">
+<attribute name="WEBLINK" value="https://lcsc.com/product-detail/PMIC-Battery-Management_UMW-Youtai-Semiconductor-Co-Ltd-TP4056_C725790.html"/>
+</part>
+<part name="Q1" library="FS8205A" deviceset="FS8205A" device="">
+<attribute name="WEBLINK" value="https://lcsc.com/product-detail/MOSFET_FUXINSEMI-FS8205A_C908265.html"/>
+</part>
+<part name="IC2" library="DW01A" deviceset="DW01A" device="">
+<attribute name="WEBLINK" value="https://lcsc.com/product-detail/Battery-Protection-ICs_PUOLOP-DW01A_C351410.html"/>
+</part>
 <part name="FRAME1" library="frames" library_urn="urn:adsk.eagle:library:229" deviceset="DINA4_L" device=""/>
 <part name="FRAME2" library="frames" library_urn="urn:adsk.eagle:library:229" deviceset="DINA4_L" device=""/>
@@
 <part name="P+6" library="supply1" library_urn="urn:adsk.eagle:library:371" deviceset="VCC" device="" value="VBAT"/>
 <part name="P+7" library="supply1" library_urn="urn:adsk.eagle:library:371" deviceset="VCC" device="" value="VIN"/>
-<part name="U1" library="SparkFun-IC-Power" library_urn="urn:adsk.eagle:library:526" deviceset="MAX1704X" device="" package3d_urn="urn:adsk.eagle:package:39055/1" value="MAX17043"/>
+<part name="U1" library="SparkFun-IC-Power" library_urn="urn:adsk.eagle:library:526" deviceset="MAX1704X" device="" package3d_urn="urn:adsk.eagle:package:39055/1" value="MAX17043">
+<attribute name="WEBLINK" value="https://www.mouser.com/ProductDetail/Maxim-Integrated/MAX17043G%2bT?qs=fnYUjNMxfVCghHGFBrnbRA%3D%3D"/>
+</part>
 <part name="C6" library="rcl" library_urn="urn:adsk.eagle:library:334" deviceset="C-EU" device="C0805" package3d_urn="urn:adsk.eagle:package:23617/2" value="1uF"/>
 <part name="R7" library="rcl" library_urn="urn:adsk.eagle:library:334" deviceset="R-US_" device="R0805" package3d_urn="urn:adsk.eagle:package:23553/2" value="180"/>
@@
 <part name="P+10" library="supply1" library_urn="urn:adsk.eagle:library:371" deviceset="VCC" device="" value="VIN"/>
 <part name="P+11" library="supply1" library_urn="urn:adsk.eagle:library:371" deviceset="VCC" device="" value="3.3V"/>
-<part name="IC3" library="DS3231" deviceset="DS3231" device="/SO"/>
+<part name="IC3" library="DS3231" deviceset="DS3231" device="/SO">
+<attribute name="WEBLINK" value="https://www.mouser.com/ProductDetail/Maxim-Integrated/DS3231SN?qs=1eQvB6Dk1vhUlr8%2FOrV0Fw%3D%3D"/>
+</part>
 <part name="P+15" library="supply1" library_urn="urn:adsk.eagle:library:371" deviceset="VCC" device="" value="3.3V"/>
 <part name="B1" library="microbuilder" deviceset="BATTERY" device="CR1220_SMT" value="CR1220"/>
 <part name="GND20" library="supply1" library_urn="urn:adsk.eagle:library:371" deviceset="GND" device=""/>
 <part name="GND21" library="supply1" library_urn="urn:adsk.eagle:library:371" deviceset="GND" device=""/>
-<part name="U4" library="SparkFun-Sensors" deviceset="ICM-20948" device="" value="9DoF IMU"/>
+<part name="U4" library="SparkFun-Sensors" deviceset="ICM-20948" device="" value="9DoF IMU">
+<attribute name="WEBLINK" value="https://www.mouser.com/ProductDetail/TDK-InvenSense/ICM-20948?qs=%2Fha2pyFaduhVfJfZCXoikyvvC70YiWC%2FBNr%2FvcBEr1bv7usabPFmkg%3D%3D"/>
+</part>
 <part name="U$1" library="SparkFun-IC-Power" library_urn="urn:adsk.eagle:library:526" deviceset="V_REG_SP6214" device="-1.8V" package3d_urn="urn:adsk.eagle:package:39079/1" value="LD39015M18R">
 <attribute name="WEBLINK" value="https://www.mouser.com/ProductDetail/STMicroelectronics/LD39015M18R?qs=%2Fha2pyFaduiNd%2F2UEBkaLCKjQ2zo%2FZOF5RG39Zh4PEGsBkDRy2IG8Q%3D%3D"/>
@@
 <part name="P+8" library="supply1" library_urn="urn:adsk.eagle:library:371" deviceset="VCC" device="" value="3.3Vesp"/>
 <part name="P+9" library="supply1" library_urn="urn:adsk.eagle:library:371" deviceset="VCC" device="" value="VIN"/>
-<part name="U5" library="ESP32-WROOM-32D" library_urn="urn:adsk.eagle:library:27379448" deviceset="ESP32-WROOM-32D" device="" package3d_urn="urn:adsk.eagle:package:27379451/1"/>
+<part name="U5" library="ESP32-WROOM-32D" library_urn="urn:adsk.eagle:library:27379448" deviceset="ESP32-WROOM-32D" device="" package3d_urn="urn:adsk.eagle:package:27379451/1">
+<attribute name="WEBLINK" value="https://www.mouser.com/ProductDetail/Espressif-Systems/ESP32-WROOM-32DM113DH2800PH3Q0?qs=W%2FMpXkg%252BdQ75%2Fda1rSxxJw%3D%3D"/>
+</part>
 <part name="J4" library="SparkFun-Connectors" deviceset="USB_MINI-B" device="_SMT" value="USB_MINI"/>
 <part name="GND36" library="supply1" library_urn="urn:adsk.eagle:library:371" deviceset="GND" device=""/>
@@
 <part name="P+37" library="supply1" library_urn="urn:adsk.eagle:library:371" deviceset="VCC" device="" value="3.3Vesp"/>
 <part name="P+38" library="supply1" library_urn="urn:adsk.eagle:library:371" deviceset="VCC" device="" value="3.3Vesp"/>
-<part name="LS1" library="CST-931AP" library_urn="urn:adsk.eagle:library:27396256" deviceset="CST-931AP" device="" package3d_urn="urn:adsk.eagle:package:27396259/1"/>
+<part name="LS1" library="CST-931AP" library_urn="urn:adsk.eagle:library:27396256" deviceset="CST-931AP" device="" package3d_urn="urn:adsk.eagle:package:27396259/1">
+<attribute name="WEBLINK" value="https://www.mouser.com/ProductDetail/CUI-Devices/CST-931AP?qs=%2Fha2pyFaduj6eTmTDzk5Y%252BDzNxLCOqaa7w%2F7LdfrL8e2VfyymTz68w%3D%3D"/>
+</part>
 <part name="Q7" library="SparkFun-DiscreteSemi" deviceset="MOSFET-NCH" device="-AO3404A" value="RUC002N05HZGT116">
 <attribute name="WEBLINK" value="https://www.mouser.com/ProductDetail/ROHM-Semiconductor/RUC002N05HZGT116?qs=4v%252BiZTmLVHE0lwSK%2FDyNsA%3D%3D"/>
@@
 <attribute name="NAME" x="27.9406" y="170.1793" size="1.27006875" layer="95" rot="R180"/>
 <attribute name="VALUE" x="38.10408125" y="144.7596" size="1.272040625" layer="96"/>
+<attribute name="WEBLINK" x="35.56" y="157.48" size="1.778" layer="96" display="off"/>
 </instance>
 <instance part="Q1" gate="G$1" x="114.3" y="142.24" smashed="yes" rot="R270">
 <attribute name="VALUE" x="107.95" y="134.62" size="1.778" layer="96"/>
 <attribute name="NAME" x="107.95" y="137.16" size="1.778" layer="95"/>
+<attribute name="WEBLINK" x="114.3" y="142.24" size="1.778" layer="96" rot="R270" display="off"/>
 </instance>
 <instance part="IC2" gate="G$1" x="88.9" y="157.48" smashed="yes">
 <attribute name="NAME" x="83.82" y="168.91" size="1.778" layer="95"/>
 <attribute name="VALUE" x="83.82" y="144.78" size="1.778" layer="95"/>
+<attribute name="WEBLINK" x="88.9" y="157.48" size="1.778" layer="96" display="off"/>
 </instance>
 <instance part="FRAME1" gate="G$1" x="0" y="0" smashed="yes"/>
@@
 <attribute name="NAME" x="226.06" y="160.274" size="1.778" layer="95"/>
 <attribute name="VALUE" x="226.06" y="142.748" size="1.778" layer="96"/>
+<attribute name="WEBLINK" x="233.68" y="152.4" size="1.778" layer="96" display="off"/>
 </instance>
 <instance part="C6" gate="G$1" x="210.82" y="147.32" smashed="yes">
@@
 <instance part="IC3" gate="G$1" x="99.06" y="109.22" smashed="yes">
 <attribute name="NAME" x="109.22" y="124.46" size="1.778" layer="95" rot="R180"/>
+<attribute name="WEBLINK" x="99.06" y="109.22" size="1.778" layer="96" display="off"/>
 </instance>
 <instance part="P+15" gate="VCC" x="78.74" y="121.92" smashed="yes">
@@
 <attribute name="NAME" x="182.88" y="68.834" size="1.778" layer="95" font="vector"/>
 <attribute name="VALUE" x="182.88" y="50.546" size="1.778" layer="96" font="vector" align="top-left"/>
+<attribute name="WEBLINK" x="195.58" y="58.42" size="1.778" layer="96" display="off"/>
 </instance>
 <instance part="U$1" gate="G$1" x="162.56" y="101.6" smashed="yes">
@@
 <attribute name="NAME" x="36.820890625" y="29.23125" size="1.782240625" layer="95"/>
 <attribute name="VALUE" x="36.81846875" y="26.6354" size="1.78338125" layer="96"/>
+<attribute name="WEBLINK" x="33.02" y="27.94" size="1.778" layer="96" display="off"/>
 </instance>
 <instance part="Q7" gate="NMOS" x="200.66" y="93.98" smashed="yes" rot="R270">
@@
 <attribute name="NAME" x="45.9241" y="133.1945" size="1.778" layer="95"/>
 <attribute name="VALUE" x="45.6733" y="65.9319" size="1.778" layer="96"/>
+<attribute name="WEBLINK" x="60.96" y="101.6" size="1.778" layer="96" display="off"/>
 </instance>
 <instance part="J4" gate="G$1" x="157.48" y="134.62" smashed="yes">

Commit message: Update serendipboard_v2.sch
Parts:
- R3: WEBLINK (none) -> https://www.mouser.com/ProductDetail/Panasonic/ERA-6VEB1001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
- R6: WEBLINK (none) -> https://www.mouser.com/ProductDetail/Panasonic/ERA-6VEB2201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
Changed lines of the file:
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@@
 <part name="R2" library="rcl" library_urn="urn:adsk.eagle:library:334" deviceset="R-US_" device="R0805" package3d_urn="urn:adsk.eagle:package:23553/2" value="100"/>
 <part name="C1" library="rcl" library_urn="urn:adsk.eagle:library:334" deviceset="C-EU" device="C0805" package3d_urn="urn:adsk.eagle:package:23617/2" value="0.1uF"/>
-<part name="R3" library="rcl" library_urn="urn:adsk.eagle:library:334" deviceset="R-US_" device="R0805" package3d_urn="urn:adsk.eagle:package:23553/2" value="1k"/>
+<part name="R3" library="rcl" library_urn="urn:adsk.eagle:library:334" deviceset="R-US_" device="R0805" package3d_urn="urn:adsk.eagle:package:23553/2" value="1k">
+<spice>
+<pinmapping spiceprefix="R">
+<pinmap gate="G$1" pin="1" pinorder="1"/>
+<pinmap gate="G$1" pin="2" pinorder="2"/>
+</pinmapping>
+</spice>
+<attribute name="WEBLINK" value="https://www.mouser.com/ProductDetail/Panasonic/ERA-6VEB1001V?qs=rI7uf1IzohSck28%2FzhwuGw%3D%3D"/>
+</part>
 <part name="GND6" library="supply1" library_urn="urn:adsk.eagle:library:371" deviceset="GND" device=""/>
 <part name="C3" library="rcl" library_urn="urn:adsk.eagle:library:334" deviceset="C-EU" device="C0805" package3d_urn="urn:adsk.eagle:package:23617/2" value="10uF"/>
@@
 <part name="JP1" library="SparkFun-Jumpers" deviceset="JUMPER-SMT_3_2-NC_TRACE" device="_SILK" package3d_urn="urn:adsk.eagle:package:39289/1" value="I2C_PU"/>
 <part name="P+19" library="supply1" library_urn="urn:adsk.eagle:library:371" deviceset="VCC" device="" value="3.3V"/>
-<part name="R6" library="rcl" library_urn="urn:adsk.eagle:library:334" deviceset="R-US_" device="R0805" package3d_urn="urn:adsk.eagle:package:23553/2" value="2.2k"/>
+<part name="R6" library="rcl" library_urn="urn:adsk.eagle:library:334" deviceset="R-US_" device="R0805" package3d_urn="urn:adsk.eagle:package:23553/2" value="2.2k">
+<spice>
+<pinmapping spiceprefix="R">
+<pinmap gate="G$1" pin="1" pinorder="1"/>
+<pinmap gate="G$1" pin="2" pinorder="2"/>
+</pinmapping>
+</spice>
+<attribute name="WEBLINK" value="https://www.mouser.com/ProductDetail/Panasonic/ERA-6VEB2201V?qs=rI7uf1IzohTwRzvkINayfg%3D%3D"/>
+</part>
 <part name="R10" library="rcl" library_urn="urn:adsk.eagle:library:334" deviceset="R-US_" device="R0805" package3d_urn="urn:adsk.eagle:package:23553/2" value="2.2k"/>
 <part name="R11" library="rcl" library_urn="urn:adsk.eagle:library:334" deviceset="R-US_" device="R0805" package3d_urn="urn:adsk.eagle:package:23553/2" value="2.2k"/>
@@
 <attribute name="NAME" x="128.4986" y="158.75" size="1.778" layer="95" rot="R270"/>
 <attribute name="VALUE" x="123.698" y="158.75" size="1.778" layer="96" rot="R270"/>
+<attribute name="WEBLINK" x="127" y="154.94" size="1.778" layer="96" rot="R270" display="off"/>
 </instance>
 <instance part="GND6" gate="1" x="127" y="137.16" smashed="yes">
@@
 <attribute name="NAME" x="206.7814" y="95.25" size="1.778" layer="95" rot="R90"/>
 <attribute name="VALUE" x="211.582" y="95.25" size="1.778" layer="96" rot="R90"/>
+<attribute name="WEBLINK" x="208.28" y="99.06" size="1.778" layer="96" rot="R90" display="off"/>
 </instance>
 <instance part="R10" gate="G$1" x="236.22" y="99.06" smashed="yes" rot="R90">

Commit message: Update serendipboard_v2.sch
Parts:
- removed C21: 47pF, rcl:C-EUC0805
- added C18: 27pF, rcl:C-EUC0402
- C20: value 27pF -> 47pF; device rcl:C-EUC0805 -> rcl:C-EUC0402
- Q2: value TRANS_NPN-MMBT2222AL -> MMBT2222ALT1G; WEBLINK (none) -> https://www.mouser.com/ProductDetail/ON-Semiconductor/MMBT2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
- Q5: value 600mA/40V -> MMBT2222ALT1G; WEBLINK (none) -> https://www.mouser.com/ProductDetail/ON-Semiconductor/MMBT2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
- Q8: value (none) -> MBT3904DW1T1G; WEBLINK (none) -> https://www.mouser.com/ProductDetail/ON-Semiconductor/MBT39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
- R19, R20: value 20k -> 4.7k
- R3: WEBLINK https://www.mouser.com/ProductDetail/Panasonic/ERA-6VEB1001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 -> (none)
- R6: WEBLINK https://www.mouser.com/ProductDetail/Panasonic/ERA-6VEB2201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 -> (none)
- renumbered Q6 to Q2
Connections:
- net GND: now also C18.2, R3.1; no longer C21.2, R3.2
- net N$16: now also C18.1; no longer C20.1
- net N$21: now also C20.1; no longer C21.1
- net N$5: now also R3.2; no longer R3.1
Other:
- moved on the sheet: C20, R3

Commit message: Update serendipboard_v2.sch
Parts:
- removed R25: 27, rcl:R-US_R0805
- added R21: 27, rcl:R-US_R0603
- J4: value USB_MINI -> USB3076-XX-X_REVC; device SparkFun-Connectors:USB_MINI-B_SMT -> USB3076-30-A:USB3076-XX-X_REVC; WEBLINK (none) -> https://www.digikey.com/en/products/detail/gct/USB3076-30-A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
- R24: device rcl:R-US_R0805 -> rcl:R-US_R0603; WEBLINK (none) -> https://www.mouser.com/ProductDetail/Panasonic/ERJ-UP3F27R0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
- U2: WEBLINK (none) -> https://www.mouser.com/ProductDetail/Diodes-Incorporated/AP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
Connections:
- new net N$24: R5.2, U2.IN
- net N$16: now also R21.1; no longer R24.1
- net N$20: now also R21.2; no longer R24.2
- net N$21: now also R24.1; no longer R25.1
- net N$22: now also R24.2; no longer R25.2
- net VCC: no longer R5.2, U2.IN
Other:
- moved on the sheet: R24

Commit message: Update serendipboard_v2.sch
Parts:
- B1: WEBLINK (none) -> https://www.digikey.com/en/products/detail/keystone-electro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
- J1: WEBLINK (none) -> https://www.mouser.com/ProductDetail/SparkFun/PRT-08612?qs=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
- S1, S2, S3, S4, S5: value (none) -> KMR731NGLFS; device SparkFun-Switches:MOMENTARY-SWITCH-SPST-2-SMD-5.2MM -> KMR731NGLFS:KMR731NGLFS; WEBLINK (none) -> https://www.mouser.com/ProductDetail/CK/KMR731NGLFS?utm_med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
Connections:
- net EN: now also S2.NO; no longer S2.3, S2.4
- net GND: now also S1.COM, S3.COM, S4.COM, S5.COM; no longer S1.1, S1.2, S2.1, S2.2, S3.1, S3.2, S4.1, S4.2, S5.1, S5.2
- net GPIO15: now also S4.NO; no longer S4.3, S4.4
- net GPIO27: now also S3.NO; no longer S3.3, S3.4
- net IO0: now also S1.NO; no longer S1.3, S1.4
- net PWR: now also S5.NO; no longer S5.3, S5.4

Commit message: Update serendipboard_v2.sch
Parts:
- removed R5: 100k, rcl:R-US_R0805
- removed U3: AP2112-3.3, microbuilder:VREG_SOT23-5
- added C21, C27: 470pF, rcl:C-EUC0402
- added U7: MIC5219 3.3V, SparkFun-IC-Power:V_REG_MIC52193.3V
- U2: value AP2112-3.3 -> MIC5219 3.3V; device microbuilder:VREG_SOT23-5 -> SparkFun-IC-Power:V_REG_MIC52193.3V; WEBLINK https://www.mouser.com/ProductDetail/Diodes-Incorporated/AP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 -> https://www.mouser.com/ProductDetail/Microchip-Technology-M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
Connections:
- new net N$25: C21.1, U7.BP
- net GND: now also C21.2, C27.2, U7.GND; no longer U3.GND
- net LOAD_EN: now also U7.EN; no longer U3.EN
- net N$24: now also C8.1, C9.1, U2.OUT; no longer R5.2, U2.IN
- net N$8: now also C27.1, U2.BP; no longer R5.1, U2.EN
- net VCC: now also U2.EN, U2.IN, U7.IN, U7.OUT; no longer C8.1, C9.1, U2.OUT, U3.IN, U3.OUT
Other:
- moved on the sheet: C10, C11, C8, C9

Commit message: Update serendipboard_v2.sch
Parts:
- renumbered J1 to BATT, J2 to M1, J3 to OLED
Changed lines of the file:
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@@
 <part name="JP2" library="SparkFun-Jumpers" deviceset="JUMPER-SMT_2_NO" device="_NO-SILK" package3d_urn="urn:adsk.eagle:package:39277/1" value="ADR"/>
 <part name="GND28" library="supply1" library_urn="urn:adsk.eagle:library:371" deviceset="GND" device=""/>
-<part name="J1" library="SparkFun-Connectors" deviceset="JST_2MM_MALE" device="">
+<part name="BATT" library="SparkFun-Connectors" deviceset="JST_2MM_MALE" device="">
 <attribute name="WEBLINK" value="https://www.mouser.com/ProductDetail/SparkFun/PRT-08612?qs=%2Fha2pyFadugGfN%252BHCaZXGW86cNwiWwmm5YQ4I4yMVjEsUzHWc0S4iQ%3D%3D"/>
 </part>
@@
 <part name="P+23" library="supply1" library_urn="urn:adsk.eagle:library:371" deviceset="VCC" device="" value="3.3V"/>
 <part name="P+24" library="supply1" library_urn="urn:adsk.eagle:library:371" deviceset="VCC" device="" value="3.3V"/>
-<part name="J2" library="SparkFun-Connectors" deviceset="CONN_02" device=""/>
+<part name="M1" library="SparkFun-Connectors" deviceset="CONN_02" device=""/>
 <part name="R15" library="rcl" library_urn="urn:adsk.eagle:library:334" deviceset="R-US_" device="R0805" package3d_urn="urn:adsk.eagle:package:23553/2" value="1k"/>
 <part name="R16" library="rcl" library_urn="urn:adsk.eagle:library:334" deviceset="R-US_" device="R0805" package3d_urn="urn:adsk.eagle:package:23553/2" value="1k"/>
@@
 <part name="P+26" library="supply1" library_urn="urn:adsk.eagle:library:371" deviceset="VCC" device="" value="VBUS"/>
 <part name="P+27" library="supply1" library_urn="urn:adsk.eagle:library:371" deviceset="VCC" device="" value="3.3V"/>
-<part name="J3" library="SparkFun-Connectors" deviceset="CONN_04" device="PTH"/>
+<part name="OLED" library="SparkFun-Connectors" deviceset="CONN_04" device="PTH"/>
 <part name="P+28" library="supply1" library_urn="urn:adsk.eagle:library:371" deviceset="VCC" device="" value="3.3V"/>
 <part name="GND35" library="supply1" library_urn="urn:adsk.eagle:library:371" deviceset="GND" device=""/>
@@
 <attribute name="VALUE" x="236.22" y="48.26" size="1.778" layer="96"/>
 </instance>
-<instance part="J1" gate="G$1" x="144.78" y="12.7" smashed="yes" rot="R90">
+<instance part="BATT" gate="G$1" x="144.78" y="12.7" smashed="yes" rot="R90">
 <attribute name="NAME" x="138.938" y="10.16" size="1.778" layer="95" rot="R90"/>
 <attribute name="WEBLINK" x="144.78" y="12.7" size="1.778" layer="96" rot="R90" display="off"/>
@@
 <attribute name="VALUE" x="35.56" y="38.1" size="1.27" layer="96" rot="R180"/>
 </instance>
-<instance part="J2" gate="G$1" x="43.18" y="73.66" smashed="yes" rot="MR0">
+<instance part="M1" gate="G$1" x="43.18" y="73.66" smashed="yes" rot="MR0">
 <attribute name="VALUE" x="45.72" y="68.834" size="1.778" layer="96" font="vector" rot="MR0"/>
 <attribute name="NAME" x="45.72" y="79.248" size="1.778" layer="95" font="vector" rot="MR0"/>
@@
 <attribute name="VALUE" x="114.3" y="38.1" size="1.27" layer="96" rot="R180"/>
 </instance>
-<instance part="J3" gate="J1" x="66.04" y="66.04" smashed="yes">
+<instance part="OLED" gate="J1" x="66.04" y="66.04" smashed="yes">
 <attribute name="VALUE" x="60.96" y="58.674" size="1.778" layer="96" font="vector"/>
 <attribute name="NAME" x="60.96" y="74.168" size="1.778" layer="95" font="vector"/>
@@
 </segment>
 <segment>
-<pinref part="J3" gate="J1" pin="3"/>
+<pinref part="OLED" gate="J1" pin="3"/>
 <wire x1="71.12" y1="68.58" x2="73.66" y2="68.58" width="0.1524" layer="91"/>
 <wire x1="73.66" y1="68.58" x2="73.66" y2="58.42" width="0.1524" layer="91"/>
@@
 </segment>
 <segment>
-<pinref part="J1" gate="G$1" pin="+"/>
+<pinref part="BATT" gate="G$1" pin="+"/>
 <wire x1="149.86" y1="15.24" x2="152.4" y2="15.24" width="0.1524" layer="91"/>
 <pinref part="P+22" gate="VCC" pin="VCC"/>
 </segment>
 <segment>
-<pinref part="J2" gate="G$1" pin="2"/>
+<pinref part="M1" gate="G$1" pin="2"/>
 <pinref part="P+23" gate="VCC" pin="VCC"/>
 <wire x1="35.56" y1="76.2" x2="33.02" y2="76.2" width="0.1524" layer="91"/>
@@
 </segment>
 <segment>
-<pinref part="J3" gate="J1" pin="4"/>
+<pinref part="OLED" gate="J1" pin="4"/>
 <wire x1="71.12" y1="71.12" x2="76.2" y2="71.12" width="0.1524" layer="91"/>
 <wire x1="76.2" y1="71.12" x2="76.2" y2="76.2" width="0.1524" layer="91"/>
@@
 </segment>
 <segment>
-<pinref part="J1" gate="G$1" pin="-"/>
+<pinref part="BATT" gate="G$1" pin="-"/>
 <wire x1="149.86" y1="12.7" x2="152.4" y2="12.7" width="0.1524" layer="91"/>
 <label x="152.4" y="12.7" size="1.27" layer="95" xref="yes"/>
@@
 </segment>
 <segment>
-<pinref part="J3" gate="J1" pin="2"/>
+<pinref part="OLED" gate="J1" pin="2"/>
 <wire x1="71.12" y1="66.04" x2="76.2" y2="66.04" width="0.1524" layer="91"/>
 <label x="76.2" y="66.04" size="1.27" layer="95" xref="yes"/>
@@
 </segment>
 <segment>
-<pinref part="J3" gate="J1" pin="1"/>
+<pinref part="OLED" gate="J1" pin="1"/>
 <wire x1="71.12" y1="63.5" x2="76.2" y2="63.5" width="0.1524" layer="91"/>
 <label x="76.2" y="63.5" size="1.27" layer="95" xref="yes"/>
@@
 <segment>
 <pinref part="Q5" gate="G$1" pin="C"/>
-<pinref part="J2" gate="G$1" pin="1"/>
+<pinref part="M1" gate="G$1" pin="1"/>
 <wire x1="33.02" y1="71.12" x2="33.02" y2="73.66" width="0.1524" layer="91"/>
 <wire x1="33.02" y1="73.66" x2="35.56" y2="73.66" width="0.1524" layer="91"/>

Commit message: .
Parts:
- added R5: 100k, rcl:R-US_R0402
- C1, C10, C11, C12, C13, C14, C15, C16, C17, C19, C2, C22, C23, C24, C25, C26, C3, C4, C5, C6, C7, C8, C9: device rcl:C-EUC0805 -> rcl:C-EUC0402
- LS1: WEBLINK https://www.mouser.com/ProductDetail/CUI-Devices/CST-931AP?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 -> (none)
- R1, R10, R11, R12, R13, R14, R15, R16, R17, R18, R19, R2, R20, R22, R23, R26, R27, R28, R3, R4, R6, R7, R8, R9: device rcl:R-US_R0805 -> rcl:R-US_R0402
- R21, R24: device rcl:R-US_R0603 -> rcl:R-US_R0402
Connections:
- removed net N$24: C8.1, C9.1, U2.OUT
- new net 1.8V: C14.1, C15.1, Q3.G, Q7.G, R10.2, R11.2, U$1.OUT, U4.VDD, U4.VDDIO
- new net 3.3V_ESP: C8.1, C9.1, R26.2, R27.2, R28.2, U2.OUT, U5.3V3
- new net 3V3OUT: C19.1, U6.3V3OUT, U6.RESET#, U6.VCCIO
- new net VBAT: BATT.+, C16.1, C3.1, IC1.BAT, Q4.D, R15.1, R2.1, R8.1
- new net VBUS: C2.1, C22.1, C23.1, C24.1, D1.A, IC1.VCC, J4.VBUS, Q4.G, R17.2, R4.2, U6.VCC
- new net VIN: C4.1, C5.1, D1.C, Q4.S, R5.1, U2.IN, U7.IN
- net GND: now also S2.COM
- net N$23: now also R5.2, U2.EN; no longer C4.1, C5.1, D1.C, Q4.S
- net VCC: no longer BATT.+, C14.1, C15.1, C16.1, C19.1, C2.1, C22.1, C23.1, C24.1, C3.1, D1.A, IC1.BAT, IC1.VCC, J4.VBUS, Q3.G, Q4.D, Q4.G, Q7.G, R10.2, R11.2, R15.1, R17.2, R2.1, R26.2, R27.2, R28.2, R4.2, R8.1, U$1.OUT, U2.EN, U2.IN, U4.VDD, U4.VDDIO, U5.3V3, U6.3V3OUT, U6.RESET#, U6.VCC, U6.VCCIO, U7.IN
Other:
- moved on the sheet: R4
